File: pcb/WePod.kicad_pcb (KiCad board)
At the start: 2 copper layers, 61 x 81 mm, 27 parts, among them J1 Display, SW1 SW_Push, SW2 SW_Push, SW3 SW_Push, SW4 SW_Push, SW5 SW_Push, U1 MOUDLE-SEEEDUINO-XIAO, U2 SD Card

Commit message: Edited an Error on the 3.3v line in the pcb
Parts:
- 3.5mm Jack: renamed from ?
- C2: renamed from 10UF; value (none) -> C
- renumbered 10uf to C1, VCC to TP1, GND to TP2, BAT to TP4, 3.3k to ´3.3k
Connections:
- J1 pad 6: VCC -> Net-(J1-Pin_1)
Routing:
- net VCC: track 124.5 -> 49.0 mm
- net Net-(J1-Pin_1): track 151.1 -> 164.8 mm
Changed lines of the file:
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@@
 			(outputformat 1)
 			(mirror no)
-			(drillshape 1)
+			(drillshape 0)
 			(scaleselection 1)
-			(outputdirectory "")
+			(outputdirectory "C:/Users/-.-/Desktop/Bambu Lab Stuff/Gerberstuff/")
 		)
 	)
@@
 			(at 0 3.75 0)
 			(layer "F.Fab")
+			(hide yes)
 			(effects
 				(font
@@
 		(descr "CP, Radial series, Radial, pin pitch=2.50mm, diameter=5mm, height=7mm, Electrolytic Capacitor")
 		(tags "CP Radial series Radial pin pitch 2.50mm diameter 5mm height 7mm Electrolytic Capacitor")
-		(property "Reference" "10uf"
+		(property "Reference" "C1"
 			(at 1.205112 0 0)
 			(layer "F.SilkS")
@@
 			(at 0 3.75 0)
 			(layer "F.Fab")
+			(hide yes)
 			(effects
 				(font
@@
 		(descr "SMD rectangular pad as test Point, square 1.0mm side length")
 		(tags "test point SMD pad rectangle square")
-		(property "Reference" "VCC"
+		(property "Reference" "TP1"
 			(at -2.5 0 0)
 			(layer "F.SilkS")
@@
 		(descr "CP, Radial series, Radial, pin pitch=2.50mm, diameter=5mm, height=7mm, Electrolytic Capacitor")
 		(tags "CP Radial series Radial pin pitch 2.50mm diameter 5mm height 7mm Electrolytic Capacitor")
-		(property "Reference" "10UF"
+		(property "Reference" "C2"
 			(at 1.205112 0 0)
 			(layer "F.SilkS")
@@
 			)
 		)
-		(property "Value" ""
+		(property "Value" "C"
 			(at 1.25 3.75 0)
 			(layer "F.Fab")
@@
 			(layers "*.Cu" "*.Mask")
 			(remove_unused_layers no)
-			(net "VCC")
+			(net "Net-(J1-Pin_1)")
 			(pinfunction "Pin_6_6")
 			(pintype "passive")
@@
 			(net "unconnected-(U1-PA8_A4_D4_SDA-Pad5)")
 			(pinfunction "PA8_A4_D4_SDA_5")
-			(pintype "passive")
+			(pintype "passive+no_connect")
 		)
 		(pad "6" thru_hole oval
@@
 			(net "unconnected-(U1-PA9_A5_D5_SCL-Pad6)")
 			(pinfunction "PA9_A5_D5_SCL_6")
-			(pintype "passive")
+			(pintype "passive+no_connect")
 		)
 		(pad "7" thru_hole oval
@@
 			(net "unconnected-(U1-PA5_A9_D9_MISO-Pad10)")
 			(pinfunction "PA5_A9_D9_MISO_10")
-			(pintype "passive")
+			(pintype "passive+no_connect")
 		)
 		(pad "11" thru_hole oval
@@
 		(descr "SMD rectangular pad as test Point, square 1.0mm side length")
 		(tags "test point SMD pad rectangle square")
-		(property "Reference" "GND"
+		(property "Reference" "TP2"
 			(at -2.5 -0.05 0)
 			(layer "F.SilkS")
@@
 			(at 0 3.75 0)
 			(layer "F.Fab")
+			(hide yes)
 			(effects
 				(font
@@
 		(descr "SMD rectangular pad as test Point, square 1.0mm side length")
 		(tags "test point SMD pad rectangle square")
-		(property "Reference" "BAT"
+		(property "Reference" "TP4"
 			(at 2.5 0 0)
 			(layer "F.SilkS")
@@
 			(at 0 3.75 0)
 			(layer "F.Fab")
+			(hide yes)
 			(effects
 				(font
@@
 		(descr "Resistor, Axial_DIN0207 series, Axial, Horizontal, pin pitch=10.16mm, 0.25W = 1/4W, length*diameter=6.3*2.5mm^2, http://cdn-reichelt.de/documents/datenblatt/B400/1_4W%23YAG.pdf")
 		(tags "Resistor Axial_DIN0207 series Axial Horizontal pin pitch 10.16mm 0.25W = 1/4W length 6.3mm diameter 2.5mm")
-		(property "Reference" "3.3k"
-			(at 5.08 0 0)
+		(property "Reference" "´3.3k"
+			(at 5.28 0 0)
 			(layer "B.SilkS")
 			(effects
@@
 		)
 		(fp_text user "${REFERENCE}"
-			(at 5.079999 0 0)
+			(at 5.28 0 0)
 			(layer "B.Fab")
 			(effects
@@
 		(descr "TRS 3.5mm, horizontal, through-hole, https://www.cuidevices.com/product/resource/pdf/sj1-352xn.pdf")
 		(tags "TRS audio jack stereo horizontal")
-		(property "Reference" ""
-			(at 0 8.8 0)
+		(property "Reference" "3.5mm Jack"
+			(at 0 1.5 0)
 			(layer "B.SilkS")
 			(effects
@@
 			(net "unconnected-(U2-SPK1-Pad6)")
 			(pinfunction "SPK1_6")
-			(pintype "passive")
+			(pintype "passive+no_connect")
 			(solder_mask_margin 0.102)
 		)
@@
 			(net "unconnected-(U2-SPK2-Pad8)")
 			(pinfunction "SPK2_8")
-			(pintype "passive")
+			(pintype "passive+no_connect")
 			(solder_mask_margin 0.102)
 		)
@@
 			(net "unconnected-(U2-IO1-Pad9)")
 			(pinfunction "IO1_9")
-			(pintype "bidirectional")
+			(pintype "bidirectional+no_connect")
 			(solder_mask_margin 0.102)
 		)
@@
 			(net "unconnected-(U2-IO2-Pad11)")
 			(pinfunction "IO2_11")
-			(pintype "bidirectional")
+			(pintype "bidirectional+no_connect")
 			(solder_mask_margin 0.102)
 		)
@@
 			(net "unconnected-(U2-ADKEY1-Pad12)")
 			(pinfunction "ADKEY1_12")
-			(pintype "input")
+			(pintype "input+no_connect")
 			(solder_mask_margin 0.102)
 		)
@@
 			(net "unconnected-(U2-ADKEY2-Pad13)")
 			(pinfunction "ADKEY2_13")
-			(pintype "input")
+			(pintype "input+no_connect")
 			(solder_mask_margin 0.102)
 		)
@@
 			(net "unconnected-(U2-USB+-Pad14)")
 			(pinfunction "USB+_14")
-			(pintype "input")
+			(pintype "input+no_connect")
 			(solder_mask_margin 0.102)
 		)
@@
 			(net "unconnected-(U2-USB--Pad15)")
 			(pinfunction "USB-_15")
-			(pintype "input")
+			(pintype "input+no_connect")
 			(solder_mask_margin 0.102)
 		)
@@
 			(net "unconnected-(U2-BUSY-Pad16)")
 			(pinfunction "BUSY_16")
-			(pintype "input")
+			(pintype "input+no_connect")
 			(solder_mask_margin 0.102)
 		)
@@
 	)
 	(segment
+		(start 128.45 51.15)
+		(end 138.85 51.15)
+		(width 0.2)
+		(layer "B.Cu")
+		(net "Net-(J1-Pin_1)")
+	)
+	(segment
 		(start 160.55 61.95)
 		(end 159.25 63.25)
@@
 	)
 	(segment
+		(start 127.3 50)
+		(end 128.45 51.15)
+		(width 0.2)
+		(layer "B.Cu")
+		(net "Net-(J1-Pin_1)")
+	)
+	(segment
 		(start 152.75 70.75)
 		(end 159.25 70.75)
@@
 	)
 	(segment
+		(start 138.85 51.15)
+		(end 140 50)
+		(width 0.2)
+		(layer "B.Cu")
+		(net "Net-(J1-Pin_1)")
+	)
+	(segment
 		(start 152.75 85.75)
 		(end 159.25 85.75)
@@
 	)
 	(segment
-		(start 127.3 50)
-		(end 128.85 48.45)
-		(width 0.2)
-		(layer "F.Cu")
-		(net "VCC")
-	)
-	(segment
 		(start 162.5 109.086346)
 		(end 162.5 108)
@@
 	)
 	(segment
-		(start 166.7 86.8)
-		(end 165.5 88)
-		(width 0.2)
-		(layer "F.Cu")
-		(net "VCC")
-	)
-	(segment
 		(start 162.5 108)
 		(end 165.5 105)
@@
 	)
 	(segment
-		(start 128.85 48.45)
-		(end 158.854164 48.45)
-		(width 0.2)
-		(layer "F.Cu")
-		(net "VCC")
-	)
-	(segment
-		(start 166.7 56.295837)
-		(end 166.7 86.8)
-		(width 0.2)
-		(layer "F.Cu")
-		(net "VCC")
-	)
-	(segment
 		(start 139.017 105.61)
 		(end 144.557 111.15)
 		(width 0.2)
 		(layer "F.Cu")
-		(net "VCC")
-	)
-	(segment
-		(start 158.854164 48.45)
-		(end 166.7 56.295837)
-		(width 0.2)
-		(layer "F.Cu")
