File: pcb/WePod.kicad_sch (KiCad schematic)
At the start: 22 parts, among them J1 Conn_01x07_Pin, J2 AudioJack3, SW1 SW_Push, SW2 SW_Push, SW3 SW_Push, SW4 SW_Push, SW5 SW_Push, U1 MOUDLE-SEEEDUINO-XIAO, U2 DFR0299

Commit message: Edited an Error on the 3.3v line in the pcb
Connections:
- net VCC: no longer J1.6 (Pin_6)
- net at J1.1 (Pin_1), R2.1, SW1.2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: now also J1.6 (Pin_6)
- no-connect marks 0 -> 12
Changed lines of the file:
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@@
+	)
+	(junction
+		(at 127 46.99)
+		(diameter 0)
+		(color 0 0 0 0)
+	)
+	(junction
+		(at 63.5 87.63)
+		(diameter 0)
+		(color 0 0 0 0)
 	)
 	(junction
@@
 	)
 	(junction
-		(at 63.5 87.63)
-		(diameter 0)
-		(color 0 0 0 0)
-	)
-	(junction
 		(at 81.28 77.47)
 		(diameter 0)
 		(color 0 0 0 0)
 	)
+	(no_connect
+		(at 104.14 111.76)
+	)
+	(no_connect
+		(at 134.62 109.22)
+	)
+	(no_connect
+		(at 104.14 96.52)
+	)
+	(no_connect
+		(at 138.43 69.85)
+	)
+	(no_connect
+		(at 97.79 69.85)
+	)
+	(no_connect
+		(at 104.14 114.3)
+	)
+	(no_connect
+		(at 104.14 99.06)
+	)
+	(no_connect
+		(at 104.14 91.44)
+	)
+	(no_connect
+		(at 104.14 104.14)
+	)
+	(no_connect
+		(at 104.14 106.68)
+	)
+	(no_connect
+		(at 97.79 72.39)
+	)
+	(no_connect
+		(at 134.62 106.68)
+	)
+	(wire
+		(pts
+			(xy 129.54 46.99) (xy 129.54 38.1)
+		)
+		(stroke
+			(width 0)
+			(type default)
+		)
+	)
 	(wire
 		(pts
@@
 	(wire
 		(pts
+			(xy 127 46.99) (xy 127 63.5)
+		)
+		(stroke
+			(width 0)
+			(type default)
+		)
+	)
+	(wire
+		(pts
 			(xy 81.28 63.5) (xy 81.28 67.31)
 		)
@@
 	(wire
 		(pts
+			(xy 115.57 38.1) (xy 115.57 45.72)
+		)
+		(stroke
+			(width 0)
+			(type default)
+		)
+	)
+	(wire
+		(pts
 			(xy 119.38 67.31) (xy 138.43 67.31)
 		)
@@
 	(wire
 		(pts
-			(xy 127 45.72) (xy 127 63.5)
+			(xy 127 45.72) (xy 127 46.99)
 		)
 		(stroke
@@
 	(wire
 		(pts
+			(xy 127 46.99) (xy 129.54 46.99)
+		)
+		(stroke
+			(width 0)
+			(type default)
+		)
+	)
+	(wire
+		(pts
 			(xy 100.33 151.13) (xy 100.33 149.86)
 		)
@@
 	(wire
 		(pts
+			(xy 115.57 45.72) (xy 114.3 45.72)
+		)
+		(stroke
+			(width 0)
+			(type default)
+		)
+	)
+	(wire
+		(pts
 			(xy 151.13 92.71) (xy 151.13 90.17)
 		)
@@
 		(pts
 			(xy 97.79 82.55) (xy 119.38 82.55)
+		)
+		(stroke
+			(width 0)
+			(type default)
+		)
+	)
+	(wire
+		(pts
+			(xy 129.54 38.1) (xy 115.57 38.1)
 		)
 		(stroke
@@
 					(unit 1)
 				)
-			)
-		)
-	)
-	(symbol
-		(lib_id "power:VCC")
-		(at 114.3 45.72 180)
-		(unit 1)
-		(body_style 1)
-		(exclude_from_sim no)
-		(in_bom yes)
-		(on_board yes)
-		(in_pos_files yes)
-		(dnp no)
-		(fields_autoplaced yes)
-		(property "Reference" "#PWR04"
-			(at 114.3 41.91 0)
-			(hide yes)
-			(show_name no)
-			(do_not_autoplace no)
-			(effects
-				(font
-					(size 1.27 1.27)
-				)
-			)
-		)
-		(property "Value" "VCC"
-			(at 114.3 50.8 0)
-			(show_name no)
-			(do_not_autoplace no)
-			(effects
-				(font
-					(size 1.27 1.27)
-				)
-			)
-		)
-		(property "Footprint" ""
-			(at 114.3 45.72 0)
-			(hide yes)
-			(show_name no)
-			(do_not_autoplace no)
-			(effects
-				(font
-					(size 1.27 1.27)
-				)
-			)
-		)
-		(property "Datasheet" ""
-			(at 114.3 45.72 0)
-			(hide yes)
-			(show_name no)
-			(do_not_autoplace no)
-			(effects
-				(font
-					(size 1.27 1.27)
-				)
-			)
-		)
-		(property "Description" "Power symbol creates a global label with name \"VCC\""
-			(at 114.3 45.72 0)
-			(hide yes)
-			(show_name no)
-			(do_not_autoplace no)
-			(effects
-				(font
-					(size 1.27 1.27)
-				)
-			)
-		)
-		(pin "1"
-		)
-		(instances
-			(project "WePod"
-				(path "/ba240a54-71eb-406a-9974-2d84abd39dc7"
-					(reference "#PWR04")
-					(unit 1)
-				)
